File: hardware/v0.1_TACS_board/v0.1_TACS_board.kicad_pcb (KiCad board)
At the start: 2 copper layers, 42 parts, among them J1 Conn_01x01_Male, J2 Conn_01x01_Male, Q1 BC847, Q2 BC857, Q3 BC857, Q4 BC847, Q5 BC857, Q6 BC847, Q7 BC857, Q8 BC847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

Commit message: finish board TACS board, generate production files, order on jlcpcb
Parts:
- added J3: Conn_01x01_Male, TestPoint:TestPoint_Pad_D2.0mm, F.Cu at (70.2, 50.9)
- added J4: Conn_01x01_Male, TestPoint:TestPoint_Pad_D2.0mm, F.Cu at (66.1, 51.0)
- R15, R16: footprint Resistor_SMD:R_0402_1005Metric -> Resistor_SMD:R_0201_0603Metric_Pad0.64x0.40mm_HandSolder
- moved R4 193.7 mm to (71.6, 36.5)
- moved R1 193.7 mm to (71.6, 35.5), turned to 180 degrees
- moved R9 178.7 mm to (70.9, 38.0), turned to 90 degrees
- moved R12 172.9 mm to (78.4, 38.2), turned to 180 degrees
- moved Q4 167.7 mm to (74.7, 37.2), turned to -90 degrees
- moved Q8 160.9 mm to (68.4, 37.0), turned to 180 degrees
- moved R11 157.3 mm to (77.8, 39.9), turned to 180 degrees
- moved Q6 150.9 mm to (64.3, 37.0)
- moved U2 147.1 mm to (82.8, 48.4), turned to -90 degrees
- moved Q1 140.1 mm to (82.2, 37.6), turned to 180 degrees
- moved R10 135.9 mm to (73.3, 51.3), turned to -90 degrees
- moved R8 134.5 mm to (73.0, 49.7)
- moved Q7 133.6 mm to (79.3, 50.3), turned to 90 degrees
- moved R6 132.3 mm to (80.0, 40.0), turned to 180 degrees
- moved Q3 131.4 mm to (75.8, 50.3), turned to 90 degrees
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Connections:
- BT1 pad 2: GND -> -BATT
- C1 pad 2: GND -> -BATT
- C2 pad 2: GND -> -BATT
- C5 pad 2: GND -> -BATT
- C6 pad 2: GND -> -BATT
- C7 pad 1: GND -> -BATT
- D1 pad 1: GND -> -BATT
- D2 pad 2: GND -> -BATT
- Q5 pad 3: Net-(R12-Pad1) -> Net-(Q5-Pad3)
- Q6 pad 3: Net-(R12-Pad1) -> Net-(Q5-Pad3)
- Q7 pad 3: Net-(R12-Pad1) -> Net-(Q5-Pad3)
- Q8 pad 3: Net-(R12-Pad1) -> Net-(Q5-Pad3)
- R12 pad 1: Net-(R12-Pad1) -> Net-(Q5-Pad3)
- R16 pad 1: GND -> -BATT
- R2 pad 2: GND -> -BATT
- R5 pad 2: Net-(R12-Pad1) -> Net-(Q5-Pad3)
- R6 pad 1: Net-(R12-Pad1) -> Net-(Q5-Pad3)
- R7 pad 2: Net-(R12-Pad1) -> Net-(Q5-Pad3)
- U1 pad 5: GND -> -BATT
- U2 pad 1: (no net) -> Net-(Q5-Pad3)
- U2 pad 2: (no net) -> -BATT
- U3 pad 2: GND -> -BATT
Routing:
- net -BATT: track 0.00 -> 72.7 mm, vias 0 -> 11
- net Net-(Q5-Pad3): track 0.00 -> 45.4 mm, vias 0 -> 2
- net +9V: track 0.00 -> 30.9 mm, vias 0 -> 4
- net Net-(Q2-Pad1): track 0.00 -> 25.4 mm, vias 0 -> 3
- net -9V: track 0.00 -> 24.3 mm, vias 0 -> 3
- net Net-(Q1-Pad3): track 0.00 -> 21.6 mm, vias 0 -> 2
- net Net-(Q1-Pad1): track 0.00 -> 21.5 mm, vias 0 -> 3
- net Net-(Q2-Pad2): track 0.00 -> 17.8 mm, vias 0 -> 2
- net /SET_V_GPIO: track 0.00 -> 16.9 mm, vias 0 -> 2
- net Net-(R15-Pad2): track 0.00 -> 13.9 mm
- net +BATT: track 0.00 -> 13.0 mm
- net Net-(Q4-Pad1): track 0.00 -> 11.6 mm
- net Net-(Q1-Pad2): track 0.00 -> 10.9 mm
- net Net-(R1-Pad2): track 0.00 -> 8.47 mm, vias 0 -> 2
- net Net-(C3-Pad2): track 0.00 -> 8.25 mm
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Other:
- board outline added: 24.6 x 18.5 mm
- board text added: "+"
- board text added: "+9V"
- board text added: "-"
- board text added: "-9V"
- board text added: "CTRL_GPIO"
- board text added: "SET_V"
