File: hardware/v0.1_TACS_board/v0.1_TACS_board.kicad_sch (KiCad schematic)
At the start: 42 parts, among them J2 Conn_01x01_Male, Q1 BC847, Q3 BC857, Q4 BC847, Q5 BC857, Q7 BC857, Q8 BC847

Commit message: finish board TACS board, generate production files, order on jlcpcb
Parts:
- added J3: (no value), symbol Connector:Conn_01x01_Male
- added J4: Conn_01x01_Male, TestPoint:TestPoint_Pad_D2.0mm, symbol Connector:Conn_01x01_Male
- BT1: value (none) -> Battery_Cell; footprint (none) -> OpenSourceSmartGlasses:BatterySolderOn
- C1, C6, C7: value (none) -> 4.7uF; footprint (none) -> Capacitor_SMD:C_0402_1005Metric
- C2: value (none) -> 0.001uF; footprint (none) -> Capacitor_SMD:C_0402_1005Metric
- C3, C4: value (none) -> 1uF; footprint (none) -> Capacitor_SMD:C_0402_1005Metric
- C5: value (none) -> 10uF; footprint (none) -> Capacitor_SMD:C_0603_1608Metric
- D2, D3: value (none) -> PMEG2010EH; footprint (none) -> Diode_SMD:D_SOD-123F
- J1: value (none) -> Conn_01x01_Male; footprint (none) -> TestPoint:TestPoint_Pad_D2.0mm
- J2: footprint (none) -> TestPoint:TestPoint_Pad_D2.0mm
- L1: value (none) -> 10uH; footprint (none) -> Inductor_SMD:L_0805_2012Metric
- Q2: value (none) -> BC857; footprint (none) -> Package_TO_SOT_SMD:SOT-23
- Q6: value (none) -> BC847; footprint (none) -> Package_TO_SOT_SMD:SOT-23
- R1, R2, R3, R9: footprint (none) -> Resistor_SMD:R_0402_1005Metric
- R10, R11: value (none) -> R_Sense; footprint (none) -> Resistor_SMD:R_0402_1005Metric
- R12, R5: value (none) -> NC; footprint (none) -> Resistor_SMD:R_0805_2012Metric
- R13, R14: value (none) -> 1; footprint (none) -> Resistor_SMD:R_0402_1005Metric
- R4: value (none) -> 4.7k; footprint (none) -> Resistor_SMD:R_0402_1005Metric
- R6: value (none) -> R_bias; footprint (none) -> Resistor_SMD:R_0402_1005Metric
- R7: value (none) -> R_Bias; footprint (none) -> Resistor_SMD:R_0402_1005Metric
- R8: value (none) -> 1k; footprint (none) -> Resistor_SMD:R_0402_1005Metric
- U1: value (none) -> Opamp_Dual; footprint (none) -> Package_SO:TSSOP-8_4.4x3mm_P0.65mm
- U3: value (none) -> LT3467AES6TRPBF; footprint (none) -> Package_TO_SOT_SMD:SOT-23-6
Connections:
- net +9V: now also J3.1 (Pin_1)
- net -9V: now also J4.1 (Pin_1)
- net -BATT: now also U2.2 (R_stim); no longer U2. (R_stim)
- net at Q5.3 (C), Q6.3 (C), Q7.3 (C)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: now also U2.1 (L_Stim); no longer U2. (R_stim)
Other:
- moved on the sheet: U1C

Commit message: sans-limiter 12V kicad schematic
Parts:
- removed Q1, Q6, Q8: BC847, Package_TO_SOT_SMD:SOT-23, symbol Transistor_BJT:BC847
- removed Q2, Q5, Q7: BC857, Package_TO_SOT_SMD:SOT-23, symbol Transistor_BJT:BC857
- removed R10, R11: R_Sense, Resistor_SMD:R_0402_1005Metric, symbol Device:R_Small
- removed R6: R_bias, Resistor_SMD:R_0402_1005Metric, symbol Device:R_Small
- removed R7: R_Bias, Resistor_SMD:R_0402_1005Metric, symbol Device:R_Small
- J3: value (none) -> Conn_01x01_Male; footprint (none) -> TestPoint:TestPoint_Pad_D2.0mm
- R12, R5: value NC -> (none)
- R15, R16: footprint (none) -> Resistor_SMD:R_0201_0603Metric_Pad0.64x0.40mm_HandSolder
- R3, R8, R9: value 1k -> (none)
- U2: value (none) -> Electrodes
Other:
- note removed: "Current Limiter Neg"
- note removed: "Current Limiter Pos"
- note removed: "R_Sense = 120 Ohm R_Bias = 200k Ohm"
- note removed: "R_Sense = 60 Ohm R_Bias = 200k Ohm"
